File: TPA3122D2_Amplifier.kicad_pcb (KiCad board)
At the start: 2 copper layers, 80 x 80 mm, 51 parts, among them J1 Barrel_Jack_Switch, J2 Screw_Terminal_01x02, J3 AudioJack3, J4 Screw_Terminal_01x04, Q1 TSM480P06, SW1 SW_Push_SPDT, U1 TPA3122D2

Commit message: updated design
Parts:
- removed G***: LOGO, logos:heritage-logo
- removed JP1, JP2: Jumper_2_Open, Connector_PinHeader_2.54mm:PinHeader_1x02_P2.54mm_Vertical
- removed REF**: OSHW-Logo2_9.8x8mm_SilkScreen, Symbol:OSHW-Logo2_9.8x8mm_SilkScreen
- added SW2: PWR OFF, Button_Switch_THT:SW_E-Switch_EG1224_SPDT_Angled, F.Cu at (134.8, 56.0)
- added TP7: ~{SD}, TestPoint:TestPoint_THTPad_D2.0mm_Drill1.0mm, F.Cu at (120.8, 62.0)
- added TP8: MUTE, TestPoint:TestPoint_THTPad_D2.0mm_Drill1.0mm, F.Cu at (137.0, 66.6)
- Q1: value TSM480P06 -> AOI21357
- SW1: value SW_Push_SPDT -> MUTE
- moved SW1 54.6 mm to (151.5, 56.0), turned to 180 degrees
- moved TP2 35.4 mm to (165.2, 53.6)
- moved TP1 33.1 mm to (158.4, 53.4)
- moved R3 19.1 mm to (125.2, 72.1), turned to 90 degrees
- moved R4 10.0 mm to (141.4, 62.3), turned to -90 degrees
- moved C13 4.23 mm to (124.6, 109.2), turned to 180 degrees
- moved J2 3.40 mm to (106.0, 99.1)
- moved Q1 0.16 mm to (118.1, 123.3)
Connections:
- Q1 pad 2: /VIN2 -> /VIN1
- SW1 pad 1: unconnected-(SW1-A-Pad1) -> VCC
- SW1 pad 2: /VIN1 -> MUTE
- SW1 pad 3: /VIN2 -> unconnected-(SW1-C-Pad3)
Routing:
- net /VIN2: track 47.6 -> 0.00 mm
- net MUTE: track 31.3 -> 47.4 mm
- net ~{SD}: track 23.6 -> 37.8 mm
- net /VIN1: track 37.7 -> 29.8 mm
- net VCC: track 220.3 -> 213.8 mm
- net RIN: track 17.6 -> 18.3 mm
- net GND: vias 96 -> 123
Other:
- board text added: "Audio in"
- board text added: "Hussam Al-Hertani 10W(15W) Stereo Class D Audio Amplifier (TPA3125(2)D2 I.C.) v0.2"
- board text added: "MUTE"
- board text added: "ON (MUTED)"
- board text added: "Pwr In (9V-28V)"
- board text added: "SHUTDOWN"
- board text added: "VCC"
- board text added: "Vol ctrl"
- board text added: "~{SD}"
- board text removed: "Hussam Al-Hertani 15W + 15 W Class D Audio Amplifier (TPA3122D2 I.C.) v0.1"
