File: TPA3122D2_Amplifier.kicad_sch (KiCad schematic)
At the start: 49 parts, among them J1 Barrel_Jack_Switch, J2 Screw_Terminal_01x02, J3 AudioJack3, J4 Screw_Terminal_01x04, Q1 TSM480P06, SW1 SW_Push_SPDT, U1 TPA3122D2

Commit message: updated design
Parts:
- removed JP1, JP2: Jumper_2_Open, Connector_PinHeader_2.54mm:PinHeader_1x02_P2.54mm_Vertical, symbol Jumper:Jumper_2_Open
- removed Q1: TSM480P06, Package_TO_SOT_THT:TO-251-3_Vertical, symbol myparts:TSM480P06
- added Q1: AOI21357, Package_TO_SOT_THT:TO-251-3_Vertical, symbol myparts:AOI21357
- added SW2: PWR OFF, Button_Switch_THT:SW_E-Switch_EG1224_SPDT_Angled, symbol Switch:SW_Push_SPDT
- added TP7: ~{SD}, TestPoint:TestPoint_THTPad_D2.0mm_Drill1.0mm, symbol Connector:TestPoint
- added TP8: MUTE, TestPoint:TestPoint_THTPad_D2.0mm_Drill1.0mm, symbol Connector:TestPoint
- SW1: value SW_Push_SPDT -> MUTE
Connections:
- net GND: now also SW2.3 (C)
- net MUTE: now also SW1.2 (B), TP8.1
- net VCC: now also SW1.1 (A), Q1.3 (S)
- net VIN1: now also Q1.2 (D); no longer SW1.2 (B)
- net ~{SD}: now also SW2.2 (B), TP7.1
- net at D1.2 (A), R1.1: now also Q1.1 (G)
- net VIN2: no longer names the net of SW1.3 (C)
- no-connect marks 1 -> 2
Other:
- note added: "TPA3122/5D2 Class D filtering stage and output"
- note added: "TPA3122/5D2 Coupling caps"
- note added: "TPA3125(2)D2"
- note removed: "TPA3122D2"
- note removed: "TPA3122D2 Class D filtering stage and output"
- note removed: "TPA3122D2 Coupling caps"
- title: (none) -> 10W(15W) Stereo Class D Audio Amplifier (TPA3125(2)D2 I.C.)
- moved on the sheet: SW1
